File: boards/ci/oparroy-ci.kicad_pcb (KiCad board)
At the start: 4 copper layers, 0 parts

Commit message: design: add scripted CI board placement
Generate a reproducible 240 x 180 mm horseshoe placement from the capture map, with stale-map, containment, and overlap checks. Document the enclosure target, scan-mapping freedom, and prototype cost envelope.

Co-authored-by: Kimi Code CLI 2.2.0 (kimi-code/k3-256k, effort: high) <noreply@moonshot.ai>
Parts:
- added BZ1: PKLCS1212E4001-R1, Buzzer_Beeper:Buzzer_Murata_PKLCS1212E, F.Cu at (52.0, 21.0)
- added BZ2: PKLCS1212E4001-R1, Buzzer_Beeper:Buzzer_Murata_PKLCS1212E, F.Cu at (162.0, 21.0)
- added BZ3: PKLCS1212E4001-R1, Buzzer_Beeper:Buzzer_Murata_PKLCS1212E, F.Cu at (188.0, 126.0)
- added C1: 100n, Capacitor_SMD:C_0603_1608Metric, F.Cu at (168.0, 82.0)
- added C10: 100n, Capacitor_SMD:C_0603_1608Metric, F.Cu at (216.0, 166.0)
- added C11: 100n, Capacitor_SMD:C_0603_1608Metric, F.Cu at (161.0, 166.0)
- added C12: 100n, Capacitor_SMD:C_0603_1608Metric, F.Cu at (106.0, 166.0)
- added C13: 100n, Capacitor_SMD:C_0603_1608Metric, F.Cu at (51.0, 166.0)
- added C14: 10u, Capacitor_SMD:C_0603_1608Metric, F.Cu at (18.0, 94.0)
- added C15: 22u, Capacitor_SMD:C_0603_1608Metric, F.Cu at (27.0, 94.0)
- added C16: 15p, Capacitor_SMD:C_0603_1608Metric, F.Cu at (56.0, 72.0)
- added C17: 15p, Capacitor_SMD:C_0603_1608Metric, F.Cu at (61.0, 72.0)
- added C18: 100n, Capacitor_SMD:C_0603_1608Metric, F.Cu at (66.0, 72.0)
- added C19: 100n, Capacitor_SMD:C_0603_1608Metric, F.Cu at (71.0, 72.0)
- added C2: 100n, Capacitor_SMD:C_0603_1608Metric, F.Cu at (180.0, 82.0)
- added C20: 100n, Capacitor_SMD:C_0603_1608Metric, F.Cu at (76.0, 72.0)
- added C21: 100n, Capacitor_SMD:C_0603_1608Metric, F.Cu at (81.0, 72.0)
- added C22: 100n, Capacitor_SMD:C_0603_1608Metric, F.Cu at (86.0, 72.0)
- added C23: 100n, Capacitor_SMD:C_0603_1608Metric, F.Cu at (56.0, 110.0)
- added C24: 100n, Capacitor_SMD:C_0603_1608Metric, F.Cu at (61.0, 110.0)
- added C25: 100n, Capacitor_SMD:C_0603_1608Metric, F.Cu at (66.0, 110.0)
- added C26: 100n, Capacitor_SMD:C_0603_1608Metric, F.Cu at (71.0, 110.0)
- added C27: 100n, Capacitor_SMD:C_0603_1608Metric, F.Cu at (76.0, 110.0)
- added C28: 1u, Capacitor_SMD:C_0603_1608Metric, F.Cu at (81.0, 110.0)
- added C29: 1u, Capacitor_SMD:C_0603_1608Metric, F.Cu at (86.0, 110.0)
- added C3: 100n, Capacitor_SMD:C_0603_1608Metric, F.Cu at (192.0, 82.0)
- added C30: 100n, Capacitor_SMD:C_0603_1608Metric, F.Cu at (33.5, 36.5)
- added C31: 10u, Capacitor_SMD:C_0603_1608Metric, F.Cu at (41.5, 36.5)
- added C32: 22n, Capacitor_SMD:C_0603_1608Metric, F.Cu at (33.0, 48.0)
- added C33: 10n, Capacitor_SMD:C_0603_1608Metric, F.Cu at (37.5, 48.0)
- added C34: 100n, Capacitor_SMD:C_0603_1608Metric, F.Cu at (88.5, 36.5)
- added C35: 10u, Capacitor_SMD:C_0603_1608Metric, F.Cu at (96.5, 36.5)
- added C36: 100n, Capacitor_SMD:C_0603_1608Metric, F.Cu at (101.0, 33.0)
- added C37: 22n, Capacitor_SMD:C_0603_1608Metric, F.Cu at (88.0, 48.0)
- added C38: 10n, Capacitor_SMD:C_0603_1608Metric, F.Cu at (92.5, 48.0)
- added C39: 100n, Capacitor_SMD:C_0603_1608Metric, F.Cu at (143.5, 36.5)
- added C4: 100n, Capacitor_SMD:C_0603_1608Metric, F.Cu at (204.0, 82.0)
- added C40: 10u, Capacitor_SMD:C_0603_1608Metric, F.Cu at (151.5, 36.5)
- added C41: 22n, Capacitor_SMD:C_0603_1608Metric, F.Cu at (143.0, 48.0)
- added C42: 10n, Capacitor_SMD:C_0603_1608Metric, F.Cu at (147.5, 48.0)
- added C43: 100n, Capacitor_SMD:C_0603_1608Metric, F.Cu at (198.5, 36.5)
- added C44: 10u, Capacitor_SMD:C_0603_1608Metric, F.Cu at (206.5, 36.5)
- added C45: 100n, Capacitor_SMD:C_0603_1608Metric, F.Cu at (211.0, 33.0)
- added C46: 22n, Capacitor_SMD:C_0603_1608Metric, F.Cu at (198.0, 48.0)
- added C47: 10n, Capacitor_SMD:C_0603_1608Metric, F.Cu at (202.5, 48.0)
- added C48: 100n, Capacitor_SMD:C_0603_1608Metric, F.Cu at (206.5, 141.5)
- added C49: 10u, Capacitor_SMD:C_0603_1608Metric, F.Cu at (198.5, 141.5)
- added C5: 100n, Capacitor_SMD:C_0603_1608Metric, F.Cu at (216.0, 82.0)
- added C50: 22n, Capacitor_SMD:C_0603_1608Metric, F.Cu at (207.0, 153.0)
- added C51: 10n, Capacitor_SMD:C_0603_1608Metric, F.Cu at (202.5, 153.0)
- added C52: 100n, Capacitor_SMD:C_0603_1608Metric, F.Cu at (151.5, 141.5)
- added C53: 10u, Capacitor_SMD:C_0603_1608Metric, F.Cu at (143.5, 141.5)
- added C54: 100n, Capacitor_SMD:C_0603_1608Metric, F.Cu at (139.0, 138.0)
- added C55: 22n, Capacitor_SMD:C_0603_1608Metric, F.Cu at (152.0, 153.0)
- added C56: 10n, Capacitor_SMD:C_0603_1608Metric, F.Cu at (147.5, 153.0)
- added C57: 100n, Capacitor_SMD:C_0603_1608Metric, F.Cu at (96.5, 141.5)
- added C58: 10u, Capacitor_SMD:C_0603_1608Metric, F.Cu at (88.5, 141.5)
- added C59: 100n, Capacitor_SMD:C_0603_1608Metric, F.Cu at (84.0, 138.0)
- added C6: 100n, Capacitor_SMD:C_0603_1608Metric, F.Cu at (24.0, 61.0)
- added C60: 1u, Capacitor_SMD:C_0603_1608Metric, F.Cu at (78.0, 138.0)
- added C61: 1n, Capacitor_SMD:C_0603_1608Metric, F.Cu at (72.0, 138.0)
- added C62: 100n, Capacitor_SMD:C_0603_1608Metric, F.Cu at (66.0, 138.0)
- added C63: 22n, Capacitor_SMD:C_0603_1608Metric, F.Cu at (97.0, 153.0)
- added C64: 10n, Capacitor_SMD:C_0603_1608Metric, F.Cu at (92.5, 153.0)
- added C65: 100n, Capacitor_SMD:C_0603_1608Metric, F.Cu at (41.5, 141.5)
- added C66: 10u, Capacitor_SMD:C_0603_1608Metric, F.Cu at (33.5, 141.5)
- added C67: 100n, Capacitor_SMD:C_0603_1608Metric, F.Cu at (29.0, 138.0)
- added C68: 22n, Capacitor_SMD:C_0603_1608Metric, F.Cu at (42.0, 153.0)
- added C69: 10n, Capacitor_SMD:C_0603_1608Metric, F.Cu at (37.5, 153.0)
- added C7: 100n, Capacitor_SMD:C_0603_1608Metric, F.Cu at (79.0, 61.0)
- added C8: 100n, Capacitor_SMD:C_0603_1608Metric, F.Cu at (134.0, 61.0)
- added C9: 100n, Capacitor_SMD:C_0603_1608Metric, F.Cu at (189.0, 61.0)
- added D1: UDD32C03L01, Diode_SMD:D_SOD-323, F.Cu at (58.0, 82.0)
- added D10: BAT54S, Package_TO_SOT_SMD:SOT-23, F.Cu at (143.5, 153.0)
- added D11: BAT54S, Package_TO_SOT_SMD:SOT-23, F.Cu at (88.5, 153.0)
- added D12: BAT54S, Package_TO_SOT_SMD:SOT-23, F.Cu at (33.5, 153.0)
- added D2: UDD32C03L01, Diode_SMD:D_SOD-323, F.Cu at (66.0, 82.0)
- added D3: UDD32C03L01, Diode_SMD:D_SOD-323, F.Cu at (21.0, 33.0)
- added D4: UDD32C03L01, Diode_SMD:D_SOD-323, F.Cu at (28.0, 33.0)
- added D5: BAT54S, Package_TO_SOT_SMD:SOT-23, F.Cu at (41.5, 48.0)
- added D6: BAT54S, Package_TO_SOT_SMD:SOT-23, F.Cu at (96.5, 48.0)
- added D7: BAT54S, Package_TO_SOT_SMD:SOT-23, F.Cu at (151.5, 48.0)
- added D8: BAT54S, Package_TO_SOT_SMD:SOT-23, F.Cu at (206.5, 48.0)
- added D9: BAT54S, Package_TO_SOT_SMD:SOT-23, F.Cu at (198.5, 153.0)
- added J1: Conn_02x05_Odd_Even, Connector_IDC:IDC-Header_2x05_P2.54mm_Vertical_SMD, F.Cu at (12.0, 75.0)
- added J2: HC-TYPE-C-16P-01A, Connector_USB:USB_C_Receptacle_HCTL_HC-TYPE-C-16P-01A, F.Cu at (5.00, 108.0)
- added J3: Conn_02x05_Odd_Even, Connector_IDC:IDC-Header_2x05_P2.54mm_Vertical_SMD, F.Cu at (14.0, 23.0)
- added LED1: XL-3216SYGC, LED_SMD:LED_1206_3216Metric, F.Cu at (13.0, 13.0)
- added LED10: XL-3216SURC, LED_SMD:LED_1206_3216Metric, F.Cu at (129.0, 13.0)
- added LED11: XL-3216SYGC, LED_SMD:LED_1206_3216Metric, F.Cu at (135.0, 13.0)
- added LED12: XL-3216UYC, LED_SMD:LED_1206_3216Metric, F.Cu at (141.0, 13.0)
- added LED13: XL-3216SYGC, LED_SMD:LED_1206_3216Metric, F.Cu at (178.0, 13.0)
- added LED14: XL-3216SURC, LED_SMD:LED_1206_3216Metric, F.Cu at (184.0, 13.0)
- added LED15: XL-3216SYGC, LED_SMD:LED_1206_3216Metric, F.Cu at (190.0, 13.0)
- added LED16: XL-3216UYC, LED_SMD:LED_1206_3216Metric, F.Cu at (196.0, 13.0)
- added LED17: XL-3216SYGC, LED_SMD:LED_1206_3216Metric, F.Cu at (227.0, 118.0)
- added LED18: XL-3216SURC, LED_SMD:LED_1206_3216Metric, F.Cu at (221.0, 118.0)
- added LED19: XL-3216SYGC, LED_SMD:LED_1206_3216Metric, F.Cu at (215.0, 118.0)
- added LED2: XL-3216SURC, LED_SMD:LED_1206_3216Metric, F.Cu at (19.0, 13.0)
- added LED20: XL-3216UYC, LED_SMD:LED_1206_3216Metric, F.Cu at (209.0, 118.0)
- added LED21: XL-3216SYGC, LED_SMD:LED_1206_3216Metric, F.Cu at (172.0, 118.0)
- added LED22: XL-3216SURC, LED_SMD:LED_1206_3216Metric, F.Cu at (166.0, 118.0)
- added LED23: XL-3216SYGC, LED_SMD:LED_1206_3216Metric, F.Cu at (160.0, 118.0)
- added LED24: XL-3216UYC, LED_SMD:LED_1206_3216Metric, F.Cu at (154.0, 118.0)
- added LED25: XL-3216SYGC, LED_SMD:LED_1206_3216Metric, F.Cu at (117.0, 118.0)
- added LED26: XL-3216SURC, LED_SMD:LED_1206_3216Metric, F.Cu at (111.0, 118.0)
- added LED27: XL-3216SYGC, LED_SMD:LED_1206_3216Metric, F.Cu at (105.0, 118.0)
- added LED28: XL-3216UYC, LED_SMD:LED_1206_3216Metric, F.Cu at (99.0, 118.0)
- added LED29: XL-3216SYGC, LED_SMD:LED_1206_3216Metric, F.Cu at (62.0, 118.0)
- added LED3: XL-3216SYGC, LED_SMD:LED_1206_3216Metric, F.Cu at (25.0, 13.0)
- added LED30: XL-3216SURC, LED_SMD:LED_1206_3216Metric, F.Cu at (56.0, 118.0)
- added LED31: XL-3216SYGC, LED_SMD:LED_1206_3216Metric, F.Cu at (50.0, 118.0)
- added LED32: XL-3216UYC, LED_SMD:LED_1206_3216Metric, F.Cu at (44.0, 118.0)
- added LED4: XL-3216UYC, LED_SMD:LED_1206_3216Metric, F.Cu at (31.0, 13.0)
- added LED5: XL-3216SYGC, LED_SMD:LED_1206_3216Metric, F.Cu at (68.0, 13.0)
- added LED6: XL-3216SURC, LED_SMD:LED_1206_3216Metric, F.Cu at (74.0, 13.0)
- added LED7: XL-3216SYGC, LED_SMD:LED_1206_3216Metric, F.Cu at (80.0, 13.0)
- added LED8: XL-3216UYC, LED_SMD:LED_1206_3216Metric, F.Cu at (86.0, 13.0)
- added LED9: XL-3216SYGC, LED_SMD:LED_1206_3216Metric, F.Cu at (123.0, 13.0)
- added Q1: AO3401A, Package_TO_SOT_SMD:SOT-23, F.Cu at (46.0, 33.0)
- added Q10: 2N7002, Package_TO_SOT_SMD:SOT-23, F.Cu at (133.0, 138.0)
- added Q11: 2N7002, Package_TO_SOT_SMD:SOT-23, F.Cu at (127.0, 138.0)
- added Q12: AO3401A, Package_TO_SOT_SMD:SOT-23, F.Cu at (121.0, 138.0)
- added Q13: AO3401A, Package_TO_SOT_SMD:SOT-23, F.Cu at (84.0, 142.0)
- added Q14: 2N7002, Package_TO_SOT_SMD:SOT-23, F.Cu at (23.0, 138.0)
- added Q15: 2N7002, Package_TO_SOT_SMD:SOT-23, F.Cu at (17.0, 138.0)
- added Q16: AO3401A, Package_TO_SOT_SMD:SOT-23, F.Cu at (11.0, 138.0)
- added Q2: 2N7002, Package_TO_SOT_SMD:SOT-23, F.Cu at (107.0, 33.0)
- added Q3: 2N7002, Package_TO_SOT_SMD:SOT-23, F.Cu at (113.0, 33.0)
- added Q4: AO3401A, Package_TO_SOT_SMD:SOT-23, F.Cu at (119.0, 33.0)
- added Q5: AO3401A, Package_TO_SOT_SMD:SOT-23, F.Cu at (156.0, 33.0)
- added Q6: 2N7002, Package_TO_SOT_SMD:SOT-23, F.Cu at (217.0, 33.0)
- added Q7: 2N7002, Package_TO_SOT_SMD:SOT-23, F.Cu at (223.0, 33.0)
- added Q8: AO3401A, Package_TO_SOT_SMD:SOT-23, F.Cu at (229.0, 33.0)
- added Q9: AO3401A, Package_TO_SOT_SMD:SOT-23, F.Cu at (194.0, 138.0)
- added R1: 47k, Resistor_SMD:R_0603_1608Metric, F.Cu at (160.0, 114.0)
- added R10: 47k, Resistor_SMD:R_0603_1608Metric, F.Cu at (168.0, 102.0)
- added R100: DNP, Resistor_SMD:R_0603_1608Metric, F.Cu at (21.0, 48.0)
- added R101: 0R, Resistor_SMD:R_0603_1608Metric, F.Cu at (28.0, 48.0)
- added R102: 10k, Resistor_SMD:R_0603_1608Metric, F.Cu at (14.0, 53.0)
- added R103: 10k, Resistor_SMD:R_0603_1608Metric, F.Cu at (21.0, 53.0)
- added R104: 470, Resistor_SMD:R_0603_1608Metric, F.Cu at (14.0, 33.5)
- added R105: 1k, Resistor_SMD:R_0603_1608Metric, F.Cu at (37.0, 13.0)
- added R106: 470, Resistor_SMD:R_0603_1608Metric, F.Cu at (43.0, 13.0)
- added R107: 1k, Resistor_SMD:R_0603_1608Metric, F.Cu at (49.0, 13.0)
- added R108: 47k, Resistor_SMD:R_0603_1608Metric, F.Cu at (33.0, 53.0)
- added R109: 220, Resistor_SMD:R_0603_1608Metric, F.Cu at (37.5, 53.0)
- added R11: 47k, Resistor_SMD:R_0603_1608Metric, F.Cu at (168.0, 105.5)
- added R110: 470, Resistor_SMD:R_0603_1608Metric, F.Cu at (101.0, 37.0)
- added R111: 470, Resistor_SMD:R_0603_1608Metric, F.Cu at (107.0, 37.0)
- added R112: 47k, Resistor_SMD:R_0603_1608Metric, F.Cu at (113.0, 37.0)
- added R113: 47k, Resistor_SMD:R_0603_1608Metric, F.Cu at (119.0, 37.0)
- added R114: 470, Resistor_SMD:R_0603_1608Metric, F.Cu at (101.0, 41.0)
- added R115: 470, Resistor_SMD:R_0603_1608Metric, F.Cu at (107.0, 41.0)
- added R116: 47k, Resistor_SMD:R_0603_1608Metric, F.Cu at (113.0, 41.0)
- added R117: 10k, Resistor_SMD:R_0603_1608Metric, F.Cu at (119.0, 41.0)
- added R118: 47k, Resistor_SMD:R_0603_1608Metric, F.Cu at (101.0, 45.0)
- added R119: 470, Resistor_SMD:R_0603_1608Metric, F.Cu at (69.0, 38.0)
- added R12: 47k, Resistor_SMD:R_0603_1608Metric, F.Cu at (168.0, 109.0)
- added R120: 470, Resistor_SMD:R_0603_1608Metric, F.Cu at (83.0, 38.0)
- added R121: 470, Resistor_SMD:R_0603_1608Metric, F.Cu at (69.0, 43.0)
- added R122: 470, Resistor_SMD:R_0603_1608Metric, F.Cu at (83.0, 43.0)
- added R123: DNP, Resistor_SMD:R_0603_1608Metric, F.Cu at (76.0, 48.0)
- added R124: 0R, Resistor_SMD:R_0603_1608Metric, F.Cu at (83.0, 48.0)
- added R125: 10k, Resistor_SMD:R_0603_1608Metric, F.Cu at (69.0, 53.0)
- added R126: 10k, Resistor_SMD:R_0603_1608Metric, F.Cu at (76.0, 53.0)
- added R127: 10k, Resistor_SMD:R_0603_1608Metric, F.Cu at (69.0, 33.5)
- added R128: 10k, Resistor_SMD:R_0603_1608Metric, F.Cu at (75.0, 33.5)
- added R129: 1k, Resistor_SMD:R_0603_1608Metric, F.Cu at (81.0, 33.5)
- added R13: 47k, Resistor_SMD:R_0603_1608Metric, F.Cu at (168.0, 112.5)
- added R130: 1k, Resistor_SMD:R_0603_1608Metric, F.Cu at (87.0, 33.5)
- added R131: 1k, Resistor_SMD:R_0603_1608Metric, F.Cu at (93.0, 33.5)
- added R132: 1k, Resistor_SMD:R_0603_1608Metric, F.Cu at (92.0, 13.0)
- added R133: 470, Resistor_SMD:R_0603_1608Metric, F.Cu at (98.0, 13.0)
- added R134: 1k, Resistor_SMD:R_0603_1608Metric, F.Cu at (104.0, 13.0)
- added R135: 47k, Resistor_SMD:R_0603_1608Metric, F.Cu at (88.0, 53.0)
- added R136: 220, Resistor_SMD:R_0603_1608Metric, F.Cu at (92.5, 53.0)
- added R137: 470, Resistor_SMD:R_0603_1608Metric, F.Cu at (162.0, 33.0)
- added R138: 470, Resistor_SMD:R_0603_1608Metric, F.Cu at (168.0, 33.0)
- added R139: 470, Resistor_SMD:R_0603_1608Metric, F.Cu at (174.0, 33.0)
- added R14: 47k, Resistor_SMD:R_0603_1608Metric, F.Cu at (180.0, 95.0)
- added R140: 470, Resistor_SMD:R_0603_1608Metric, F.Cu at (156.0, 37.0)
- added R141: 47k, Resistor_SMD:R_0603_1608Metric, F.Cu at (162.0, 37.0)
- added R142: 47k, Resistor_SMD:R_0603_1608Metric, F.Cu at (168.0, 37.0)
- added R143: 470, Resistor_SMD:R_0603_1608Metric, F.Cu at (124.0, 38.0)
- added R144: 470, Resistor_SMD:R_0603_1608Metric, F.Cu at (138.0, 38.0)
- added R145: 470, Resistor_SMD:R_0603_1608Metric, F.Cu at (124.0, 43.0)
- added R146: 470, Resistor_SMD:R_0603_1608Metric, F.Cu at (138.0, 43.0)
- added R147: DNP, Resistor_SMD:R_0603_1608Metric, F.Cu at (131.0, 48.0)
- added R148: 0R, Resistor_SMD:R_0603_1608Metric, F.Cu at (138.0, 48.0)
- added R149: 10k, Resistor_SMD:R_0603_1608Metric, F.Cu at (124.0, 53.0)
- added R15: 47k, Resistor_SMD:R_0603_1608Metric, F.Cu at (31.0, 61.0)
- added R150: 10k, Resistor_SMD:R_0603_1608Metric, F.Cu at (131.0, 53.0)
- added R151: 470, Resistor_SMD:R_0603_1608Metric, F.Cu at (124.0, 33.5)
- added R152: 1k, Resistor_SMD:R_0603_1608Metric, F.Cu at (147.0, 13.0)
- added R153: 470, Resistor_SMD:R_0603_1608Metric, F.Cu at (153.0, 13.0)
- added R154: 1k, Resistor_SMD:R_0603_1608Metric, F.Cu at (159.0, 13.0)
- added R155: 47k, Resistor_SMD:R_0603_1608Metric, F.Cu at (143.0, 53.0)
- added R156: 220, Resistor_SMD:R_0603_1608Metric, F.Cu at (147.5, 53.0)
- added R157: 470, Resistor_SMD:R_0603_1608Metric, F.Cu at (211.0, 37.0)
- added R158: 470, Resistor_SMD:R_0603_1608Metric, F.Cu at (217.0, 37.0)
- added R159: 47k, Resistor_SMD:R_0603_1608Metric, F.Cu at (223.0, 37.0)
- added R16: 47k, Resistor_SMD:R_0603_1608Metric, F.Cu at (35.5, 61.0)
- added R160: 47k, Resistor_SMD:R_0603_1608Metric, F.Cu at (229.0, 37.0)
- added R161: 470, Resistor_SMD:R_0603_1608Metric, F.Cu at (211.0, 41.0)
- added R162: 470, Resistor_SMD:R_0603_1608Metric, F.Cu at (217.0, 41.0)
- added R163: 47k, Resistor_SMD:R_0603_1608Metric, F.Cu at (223.0, 41.0)
- added R164: 10k, Resistor_SMD:R_0603_1608Metric, F.Cu at (229.0, 41.0)
- added R165: 47k, Resistor_SMD:R_0603_1608Metric, F.Cu at (211.0, 45.0)
- added R166: 470, Resistor_SMD:R_0603_1608Metric, F.Cu at (179.0, 38.0)
- added R167: 470, Resistor_SMD:R_0603_1608Metric, F.Cu at (193.0, 38.0)
- added R168: 470, Resistor_SMD:R_0603_1608Metric, F.Cu at (179.0, 43.0)
- added R169: 470, Resistor_SMD:R_0603_1608Metric, F.Cu at (193.0, 43.0)
- added R17: 47k, Resistor_SMD:R_0603_1608Metric, F.Cu at (40.0, 61.0)
- added R170: DNP, Resistor_SMD:R_0603_1608Metric, F.Cu at (186.0, 48.0)
- added R171: 0R, Resistor_SMD:R_0603_1608Metric, F.Cu at (193.0, 48.0)
- added R172: 10k, Resistor_SMD:R_0603_1608Metric, F.Cu at (179.0, 53.0)
- added R173: 10k, Resistor_SMD:R_0603_1608Metric, F.Cu at (186.0, 53.0)
- added R174: 10k, Resistor_SMD:R_0603_1608Metric, F.Cu at (179.0, 33.5)
- added R175: 10k, Resistor_SMD:R_0603_1608Metric, F.Cu at (185.0, 33.5)
- added R176: 1k, Resistor_SMD:R_0603_1608Metric, F.Cu at (191.0, 33.5)
- added R177: 1k, Resistor_SMD:R_0603_1608Metric, F.Cu at (197.0, 33.5)
- added R178: 1k, Resistor_SMD:R_0603_1608Metric, F.Cu at (203.0, 33.5)
- added R179: 1k, Resistor_SMD:R_0603_1608Metric, F.Cu at (202.0, 13.0)
- added R18: 47k, Resistor_SMD:R_0603_1608Metric, F.Cu at (44.5, 61.0)
- added R180: 470, Resistor_SMD:R_0603_1608Metric, F.Cu at (208.0, 13.0)
- added R181: 1k, Resistor_SMD:R_0603_1608Metric, F.Cu at (214.0, 13.0)
- added R182: 47k, Resistor_SMD:R_0603_1608Metric, F.Cu at (198.0, 53.0)
- added R183: 220, Resistor_SMD:R_0603_1608Metric, F.Cu at (202.5, 53.0)
- added R184: 470, Resistor_SMD:R_0603_1608Metric, F.Cu at (188.0, 138.0)
- added R185: 470, Resistor_SMD:R_0603_1608Metric, F.Cu at (182.0, 138.0)
- added R186: 470, Resistor_SMD:R_0603_1608Metric, F.Cu at (176.0, 138.0)
- added R187: 470, Resistor_SMD:R_0603_1608Metric, F.Cu at (194.0, 142.0)
- added R188: 47k, Resistor_SMD:R_0603_1608Metric, F.Cu at (188.0, 142.0)
- added R189: 47k, Resistor_SMD:R_0603_1608Metric, F.Cu at (182.0, 142.0)
- added R19: 47k, Resistor_SMD:R_0603_1608Metric, F.Cu at (49.0, 61.0)
- added R190: 470, Resistor_SMD:R_0603_1608Metric, F.Cu at (226.0, 143.0)
- added R191: 470, Resistor_SMD:R_0603_1608Metric, F.Cu at (212.0, 143.0)
- added R192: 470, Resistor_SMD:R_0603_1608Metric, F.Cu at (226.0, 148.0)
- added R193: 470, Resistor_SMD:R_0603_1608Metric, F.Cu at (212.0, 148.0)
- added R194: DNP, Resistor_SMD:R_0603_1608Metric, F.Cu at (219.0, 153.0)
- added R195: 0R, Resistor_SMD:R_0603_1608Metric, F.Cu at (212.0, 153.0)
- added R196: 10k, Resistor_SMD:R_0603_1608Metric, F.Cu at (226.0, 158.0)
- added R197: 10k, Resistor_SMD:R_0603_1608Metric, F.Cu at (219.0, 158.0)
- added R198: 470, Resistor_SMD:R_0603_1608Metric, F.Cu at (226.0, 138.5)
- added R199: 1k, Resistor_SMD:R_0603_1608Metric, F.Cu at (203.0, 118.0)
- added R2: 47k, Resistor_SMD:R_0603_1608Metric, F.Cu at (180.0, 88.0)
- added R20: 47k, Resistor_SMD:R_0603_1608Metric, F.Cu at (53.5, 61.0)
- added R200: 470, Resistor_SMD:R_0603_1608Metric, F.Cu at (197.0, 118.0)
- added R201: 1k, Resistor_SMD:R_0603_1608Metric, F.Cu at (191.0, 118.0)
- added R202: 47k, Resistor_SMD:R_0603_1608Metric, F.Cu at (207.0, 158.0)
- added R203: 220, Resistor_SMD:R_0603_1608Metric, F.Cu at (202.5, 158.0)
- added R204: 470, Resistor_SMD:R_0603_1608Metric, F.Cu at (139.0, 142.0)
- added R205: 470, Resistor_SMD:R_0603_1608Metric, F.Cu at (133.0, 142.0)
- added R206: 47k, Resistor_SMD:R_0603_1608Metric, F.Cu at (127.0, 142.0)
- added R207: 47k, Resistor_SMD:R_0603_1608Metric, F.Cu at (121.0, 142.0)
- added R208: 470, Resistor_SMD:R_0603_1608Metric, F.Cu at (139.0, 146.0)
- added R209: 470, Resistor_SMD:R_0603_1608Metric, F.Cu at (133.0, 146.0)
- added R21: 47k, Resistor_SMD:R_0603_1608Metric, F.Cu at (58.0, 61.0)
- added R210: 47k, Resistor_SMD:R_0603_1608Metric, F.Cu at (127.0, 146.0)
- added R211: 10k, Resistor_SMD:R_0603_1608Metric, F.Cu at (121.0, 146.0)
- added R212: 47k, Resistor_SMD:R_0603_1608Metric, F.Cu at (139.0, 150.0)
- added R213: 470, Resistor_SMD:R_0603_1608Metric, F.Cu at (171.0, 143.0)
- added R214: 470, Resistor_SMD:R_0603_1608Metric, F.Cu at (157.0, 143.0)
- added R215: 470, Resistor_SMD:R_0603_1608Metric, F.Cu at (171.0, 148.0)
- added R216: 470, Resistor_SMD:R_0603_1608Metric, F.Cu at (157.0, 148.0)
- added R217: DNP, Resistor_SMD:R_0603_1608Metric, F.Cu at (164.0, 153.0)
- added R218: 0R, Resistor_SMD:R_0603_1608Metric, F.Cu at (157.0, 153.0)
- added R219: 10k, Resistor_SMD:R_0603_1608Metric, F.Cu at (171.0, 158.0)
- added R22: 47k, Resistor_SMD:R_0603_1608Metric, F.Cu at (86.0, 61.0)
- added R220: 10k, Resistor_SMD:R_0603_1608Metric, F.Cu at (164.0, 158.0)
- added R221: 10k, Resistor_SMD:R_0603_1608Metric, F.Cu at (171.0, 138.5)
- added R222: 10k, Resistor_SMD:R_0603_1608Metric, F.Cu at (165.0, 138.5)
- added R223: 1k, Resistor_SMD:R_0603_1608Metric, F.Cu at (159.0, 138.5)
- added R224: 1k, Resistor_SMD:R_0603_1608Metric, F.Cu at (153.0, 138.5)
- added R225: 1k, Resistor_SMD:R_0603_1608Metric, F.Cu at (147.0, 138.5)
- added R226: 1k, Resistor_SMD:R_0603_1608Metric, F.Cu at (148.0, 118.0)
- added R227: 470, Resistor_SMD:R_0603_1608Metric, F.Cu at (142.0, 118.0)
- added R228: 1k, Resistor_SMD:R_0603_1608Metric, F.Cu at (136.0, 118.0)
- added R229: 47k, Resistor_SMD:R_0603_1608Metric, F.Cu at (152.0, 158.0)
- added R23: 47k, Resistor_SMD:R_0603_1608Metric, F.Cu at (90.5, 61.0)
- added R230: 220, Resistor_SMD:R_0603_1608Metric, F.Cu at (147.5, 158.0)
- added R231: 47k, Resistor_SMD:R_0603_1608Metric, F.Cu at (78.0, 142.0)
- added R232: 47, Resistor_SMD:R_0603_1608Metric, F.Cu at (72.0, 142.0)
- added R233: 47k, Resistor_SMD:R_0603_1608Metric, F.Cu at (66.0, 142.0)
- added R234: R082, Resistor_SMD:R_0603_1608Metric, F.Cu at (84.0, 146.0)
- added R235: 470, Resistor_SMD:R_0603_1608Metric, F.Cu at (116.0, 143.0)
- added R236: 470, Resistor_SMD:R_0603_1608Metric, F.Cu at (102.0, 143.0)
- added R237: 470, Resistor_SMD:R_0603_1608Metric, F.Cu at (116.0, 148.0)
- added R238: 470, Resistor_SMD:R_0603_1608Metric, F.Cu at (102.0, 148.0)
- added R239: DNP, Resistor_SMD:R_0603_1608Metric, F.Cu at (109.0, 153.0)
- added R24: 47k, Resistor_SMD:R_0603_1608Metric, F.Cu at (95.0, 61.0)
- added R240: 0R, Resistor_SMD:R_0603_1608Metric, F.Cu at (102.0, 153.0)
- added R241: 10k, Resistor_SMD:R_0603_1608Metric, F.Cu at (116.0, 158.0)
- added R242: 10k, Resistor_SMD:R_0603_1608Metric, F.Cu at (109.0, 158.0)
- added R243: 1k, Resistor_SMD:R_0603_1608Metric, F.Cu at (93.0, 118.0)
- added R244: 470, Resistor_SMD:R_0603_1608Metric, F.Cu at (87.0, 118.0)
- added R245: 1k, Resistor_SMD:R_0603_1608Metric, F.Cu at (81.0, 118.0)
- added R246: 47k, Resistor_SMD:R_0603_1608Metric, F.Cu at (97.0, 158.0)
- added R247: 220, Resistor_SMD:R_0603_1608Metric, F.Cu at (92.5, 158.0)
- added R248: 470, Resistor_SMD:R_0603_1608Metric, F.Cu at (29.0, 142.0)
- added R249: 470, Resistor_SMD:R_0603_1608Metric, F.Cu at (23.0, 142.0)
- added R25: 47k, Resistor_SMD:R_0603_1608Metric, F.Cu at (99.5, 61.0)
- added R250: 47k, Resistor_SMD:R_0603_1608Metric, F.Cu at (17.0, 142.0)
- added R251: 47k, Resistor_SMD:R_0603_1608Metric, F.Cu at (11.0, 142.0)
- added R252: 470, Resistor_SMD:R_0603_1608Metric, F.Cu at (29.0, 146.0)
- added R253: 470, Resistor_SMD:R_0603_1608Metric, F.Cu at (23.0, 146.0)
- added R254: 47k, Resistor_SMD:R_0603_1608Metric, F.Cu at (17.0, 146.0)
- added R255: 10k, Resistor_SMD:R_0603_1608Metric, F.Cu at (11.0, 146.0)
- added R256: 47k, Resistor_SMD:R_0603_1608Metric, F.Cu at (29.0, 150.0)
- added R257: 470, Resistor_SMD:R_0603_1608Metric, F.Cu at (61.0, 143.0)
- added R258: 470, Resistor_SMD:R_0603_1608Metric, F.Cu at (47.0, 143.0)
- added R259: 470, Resistor_SMD:R_0603_1608Metric, F.Cu at (61.0, 148.0)
- added R26: 47k, Resistor_SMD:R_0603_1608Metric, F.Cu at (104.0, 61.0)
- added R260: 470, Resistor_SMD:R_0603_1608Metric, F.Cu at (47.0, 148.0)
- added R261: DNP, Resistor_SMD:R_0603_1608Metric, F.Cu at (54.0, 153.0)
- added R262: 0R, Resistor_SMD:R_0603_1608Metric, F.Cu at (47.0, 153.0)
- added R263: 10k, Resistor_SMD:R_0603_1608Metric, F.Cu at (61.0, 158.0)
- added R264: 10k, Resistor_SMD:R_0603_1608Metric, F.Cu at (54.0, 158.0)
- added R265: 10k, Resistor_SMD:R_0603_1608Metric, F.Cu at (61.0, 138.5)
- added R266: 10k, Resistor_SMD:R_0603_1608Metric, F.Cu at (55.0, 138.5)
- added R267: 1k, Resistor_SMD:R_0603_1608Metric, F.Cu at (49.0, 138.5)
- added R268: 1k, Resistor_SMD:R_0603_1608Metric, F.Cu at (43.0, 138.5)
- added R269: 1k, Resistor_SMD:R_0603_1608Metric, F.Cu at (37.0, 138.5)
- added R27: 47k, Resistor_SMD:R_0603_1608Metric, F.Cu at (108.5, 61.0)
- added R270: 1k, Resistor_SMD:R_0603_1608Metric, F.Cu at (38.0, 118.0)
- added R271: 470, Resistor_SMD:R_0603_1608Metric, F.Cu at (32.0, 118.0)
- added R272: 1k, Resistor_SMD:R_0603_1608Metric, F.Cu at (26.0, 118.0)
- added R273: 47k, Resistor_SMD:R_0603_1608Metric, F.Cu at (42.0, 158.0)
- added R274: 220, Resistor_SMD:R_0603_1608Metric, F.Cu at (37.5, 158.0)
- added R28: 47k, Resistor_SMD:R_0603_1608Metric, F.Cu at (113.0, 61.0)
- added R29: 47k, Resistor_SMD:R_0603_1608Metric, F.Cu at (141.0, 61.0)
- added R3: 47k, Resistor_SMD:R_0603_1608Metric, F.Cu at (180.0, 91.5)
- added R30: 47k, Resistor_SMD:R_0603_1608Metric, F.Cu at (145.5, 61.0)
- added R31: 47k, Resistor_SMD:R_0603_1608Metric, F.Cu at (150.0, 61.0)
- added R32: 47k, Resistor_SMD:R_0603_1608Metric, F.Cu at (154.5, 61.0)
- added R33: 47k, Resistor_SMD:R_0603_1608Metric, F.Cu at (159.0, 61.0)
- added R34: 47k, Resistor_SMD:R_0603_1608Metric, F.Cu at (163.5, 61.0)
- added R35: 47k, Resistor_SMD:R_0603_1608Metric, F.Cu at (168.0, 61.0)
- added R36: 47k, Resistor_SMD:R_0603_1608Metric, F.Cu at (196.0, 61.0)
- added R37: 47k, Resistor_SMD:R_0603_1608Metric, F.Cu at (200.5, 61.0)
- added R38: 47k, Resistor_SMD:R_0603_1608Metric, F.Cu at (205.0, 61.0)
- added R39: 47k, Resistor_SMD:R_0603_1608Metric, F.Cu at (209.5, 61.0)
- added R4: 47k, Resistor_SMD:R_0603_1608Metric, F.Cu at (192.0, 88.0)
- added R40: 47k, Resistor_SMD:R_0603_1608Metric, F.Cu at (214.0, 61.0)
- added R41: 47k, Resistor_SMD:R_0603_1608Metric, F.Cu at (218.5, 61.0)
- added R42: 47k, Resistor_SMD:R_0603_1608Metric, F.Cu at (223.0, 61.0)
- added R43: 47k, Resistor_SMD:R_0603_1608Metric, F.Cu at (209.0, 166.0)
- added R44: 47k, Resistor_SMD:R_0603_1608Metric, F.Cu at (204.5, 166.0)
- added R45: 47k, Resistor_SMD:R_0603_1608Metric, F.Cu at (200.0, 166.0)
- added R46: 47k, Resistor_SMD:R_0603_1608Metric, F.Cu at (195.5, 166.0)
- added R47: 47k, Resistor_SMD:R_0603_1608Metric, F.Cu at (191.0, 166.0)
- added R48: 47k, Resistor_SMD:R_0603_1608Metric, F.Cu at (186.5, 166.0)
- added R49: 47k, Resistor_SMD:R_0603_1608Metric, F.Cu at (182.0, 166.0)
- added R5: 47k, Resistor_SMD:R_0603_1608Metric, F.Cu at (192.0, 91.5)
- added R50: 47k, Resistor_SMD:R_0603_1608Metric, F.Cu at (154.0, 166.0)
- added R51: 47k, Resistor_SMD:R_0603_1608Metric, F.Cu at (149.5, 166.0)
- added R52: 47k, Resistor_SMD:R_0603_1608Metric, F.Cu at (145.0, 166.0)
- added R53: 47k, Resistor_SMD:R_0603_1608Metric, F.Cu at (140.5, 166.0)
- added R54: 47k, Resistor_SMD:R_0603_1608Metric, F.Cu at (136.0, 166.0)
- added R55: 47k, Resistor_SMD:R_0603_1608Metric, F.Cu at (131.5, 166.0)
- added R56: 47k, Resistor_SMD:R_0603_1608Metric, F.Cu at (127.0, 166.0)
- added R57: 47k, Resistor_SMD:R_0603_1608Metric, F.Cu at (44.0, 166.0)
- added R58: 47k, Resistor_SMD:R_0603_1608Metric, F.Cu at (39.5, 166.0)
- added R59: 47k, Resistor_SMD:R_0603_1608Metric, F.Cu at (35.0, 166.0)
- added R6: 47k, Resistor_SMD:R_0603_1608Metric, F.Cu at (168.0, 88.0)
- added R60: 47k, Resistor_SMD:R_0603_1608Metric, F.Cu at (30.5, 166.0)
- added R61: 47k, Resistor_SMD:R_0603_1608Metric, F.Cu at (26.0, 166.0)
- added R62: 47k, Resistor_SMD:R_0603_1608Metric, F.Cu at (21.5, 166.0)
- added R63: 47k, Resistor_SMD:R_0603_1608Metric, F.Cu at (17.0, 166.0)
- added R64: 47k, Resistor_SMD:R_0603_1608Metric, F.Cu at (180.0, 98.5)
- added R65: 5k1, Resistor_SMD:R_0603_1608Metric, F.Cu at (18.0, 111.0)
- added R66: 5k1, Resistor_SMD:R_0603_1608Metric, F.Cu at (27.0, 111.0)
- added R67: 470, Resistor_SMD:R_0603_1608Metric, F.Cu at (34.0, 72.0)
- added R68: 470, Resistor_SMD:R_0603_1608Metric, F.Cu at (40.0, 72.0)
- added R69: 470, Resistor_SMD:R_0603_1608Metric, F.Cu at (46.0, 72.0)
- added R7: 47k, Resistor_SMD:R_0603_1608Metric, F.Cu at (168.0, 91.5)
- added R70: 470, Resistor_SMD:R_0603_1608Metric, F.Cu at (34.0, 80.0)
- added R71: 1k, Resistor_SMD:R_0603_1608Metric, F.Cu at (74.0, 82.0)
- added R72: 10k, Resistor_SMD:R_0603_1608Metric, F.Cu at (82.0, 82.0)
- added R73: 1k, Resistor_SMD:R_0603_1608Metric, F.Cu at (58.0, 98.0)
- added R74: 27, Resistor_SMD:R_0603_1608Metric, F.Cu at (66.0, 98.0)
- added R75: 27, Resistor_SMD:R_0603_1608Metric, F.Cu at (74.0, 98.0)
- added R76: 470, Resistor_SMD:R_0603_1608Metric, F.Cu at (82.0, 98.0)
- added R77: 470, Resistor_SMD:R_0603_1608Metric, F.Cu at (58.0, 113.0)
- added R78: 470, Resistor_SMD:R_0603_1608Metric, F.Cu at (66.0, 113.0)
- added R79: 470, Resistor_SMD:R_0603_1608Metric, F.Cu at (74.0, 113.0)
- added R8: 47k, Resistor_SMD:R_0603_1608Metric, F.Cu at (168.0, 95.0)
- added R80: 10k, Resistor_SMD:R_0603_1608Metric, F.Cu at (120.0, 70.0)
- added R81: 10k, Resistor_SMD:R_0603_1608Metric, F.Cu at (120.0, 80.0)
- added R82: 10k, Resistor_SMD:R_0603_1608Metric, F.Cu at (120.0, 100.0)
- added R83: 10k, Resistor_SMD:R_0603_1608Metric, F.Cu at (120.0, 110.0)
- added R84: 10k, Resistor_SMD:R_0603_1608Metric, F.Cu at (125.0, 70.0)
- added R85: 10k, Resistor_SMD:R_0603_1608Metric, F.Cu at (125.0, 80.0)
- added R86: 10k, Resistor_SMD:R_0603_1608Metric, F.Cu at (125.0, 100.0)
- added R87: 10k, Resistor_SMD:R_0603_1608Metric, F.Cu at (125.0, 110.0)
- added R88: 4k7, Resistor_SMD:R_0603_1608Metric, F.Cu at (90.0, 104.0)
- added R89: 470, Resistor_SMD:R_0603_1608Metric, F.Cu at (52.0, 33.0)
- added R9: 47k, Resistor_SMD:R_0603_1608Metric, F.Cu at (168.0, 98.5)
- added R90: 470, Resistor_SMD:R_0603_1608Metric, F.Cu at (58.0, 33.0)
- added R91: 470, Resistor_SMD:R_0603_1608Metric, F.Cu at (64.0, 33.0)
- added R92: 470, Resistor_SMD:R_0603_1608Metric, F.Cu at (46.0, 37.0)
- added R93: 47k, Resistor_SMD:R_0603_1608Metric, F.Cu at (52.0, 37.0)
- added R94: 47k, Resistor_SMD:R_0603_1608Metric, F.Cu at (58.0, 37.0)
- added R95: 470, Resistor_SMD:R_0603_1608Metric, F.Cu at (64.0, 37.0)
- added R96: 470, Resistor_SMD:R_0603_1608Metric, F.Cu at (14.0, 38.0)
- added R97: 470, Resistor_SMD:R_0603_1608Metric, F.Cu at (28.0, 38.0)
- added R98: 470, Resistor_SMD:R_0603_1608Metric, F.Cu at (14.0, 43.0)
- added R99: 470, Resistor_SMD:R_0603_1608Metric, F.Cu at (28.0, 43.0)
- added RV1: 10k, Potentiometer_THT:Potentiometer_Alps_RK09K_Single_Vertical, F.Cu at (75.0, 23.0)
- added RV2: 10k, Potentiometer_THT:Potentiometer_Alps_RK09K_Single_Vertical, F.Cu at (185.0, 23.0)
- added RV3: 10k, Potentiometer_THT:Potentiometer_Alps_RK09K_Single_Vertical, F.Cu at (165.0, 128.0)
- added RV4: 10k, Potentiometer_THT:Potentiometer_Alps_RK09K_Single_Vertical, F.Cu at (55.0, 128.0)
- added SW1: TS-1187A-B-A-B, Button_Switch_SMD:SW_Push_1P1T_XKB_TS-1187A, F.Cu at (95.0, 23.0)
- added SW2: TS-1187A-B-A-B, Button_Switch_SMD:SW_Push_1P1T_XKB_TS-1187A, F.Cu at (110.0, 23.0)
- added SW3: TS-1187A-B-A-B, Button_Switch_SMD:SW_Push_1P1T_XKB_TS-1187A, F.Cu at (205.0, 23.0)
- added SW4: TS-1187A-B-A-B, Button_Switch_SMD:SW_Push_1P1T_XKB_TS-1187A, F.Cu at (220.0, 23.0)
- added SW5: TS-1187A-B-A-B, Button_Switch_SMD:SW_Push_1P1T_XKB_TS-1187A, F.Cu at (145.0, 128.0)
- added SW6: TS-1187A-B-A-B, Button_Switch_SMD:SW_Push_1P1T_XKB_TS-1187A, F.Cu at (130.0, 128.0)
- added SW7: TS-1187A-B-A-B, Button_Switch_SMD:SW_Push_1P1T_XKB_TS-1187A, F.Cu at (35.0, 128.0)
- added SW8: TS-1187A-B-A-B, Button_Switch_SMD:SW_Push_1P1T_XKB_TS-1187A, F.Cu at (20.0, 128.0)
- added TP1: SWIO, TestPoint:TestPoint_Pad_1.5x1.5mm, F.Cu at (38.0, 30.0)
- added TP10: 3V3, TestPoint:TestPoint_Pad_1.5x1.5mm, F.Cu at (154.0, 30.0)
- added TP11: GND, TestPoint:TestPoint_Pad_1.5x1.5mm, F.Cu at (160.0, 30.0)
- added TP12: PC7, TestPoint:TestPoint_Pad_1.5x1.5mm, F.Cu at (166.0, 30.0)
- added TP13: SWIO, TestPoint:TestPoint_Pad_1.5x1.5mm, F.Cu at (203.0, 30.0)
- added TP14: 3V3, TestPoint:TestPoint_Pad_1.5x1.5mm, F.Cu at (209.0, 30.0)
- added TP15: GND, TestPoint:TestPoint_Pad_1.5x1.5mm, F.Cu at (215.0, 30.0)
- added TP16: PC7, TestPoint:TestPoint_Pad_1.5x1.5mm, F.Cu at (221.0, 30.0)
- added TP17: SWIO, TestPoint:TestPoint_Pad_1.5x1.5mm, F.Cu at (202.0, 135.0)
- added TP18: 3V3, TestPoint:TestPoint_Pad_1.5x1.5mm, F.Cu at (196.0, 135.0)
- added TP19: GND, TestPoint:TestPoint_Pad_1.5x1.5mm, F.Cu at (190.0, 135.0)
- added TP2: 3V3, TestPoint:TestPoint_Pad_1.5x1.5mm, F.Cu at (44.0, 30.0)
- added TP20: PC7, TestPoint:TestPoint_Pad_1.5x1.5mm, F.Cu at (184.0, 135.0)
- added TP21: SWIO, TestPoint:TestPoint_Pad_1.5x1.5mm, F.Cu at (147.0, 135.0)
- added TP22: 3V3, TestPoint:TestPoint_Pad_1.5x1.5mm, F.Cu at (141.0, 135.0)
- added TP23: GND, TestPoint:TestPoint_Pad_1.5x1.5mm, F.Cu at (135.0, 135.0)
- added TP24: PC7, TestPoint:TestPoint_Pad_1.5x1.5mm, F.Cu at (129.0, 135.0)
- added TP25: SWIO, TestPoint:TestPoint_Pad_1.5x1.5mm, F.Cu at (92.0, 135.0)
- added TP26: 3V3, TestPoint:TestPoint_Pad_1.5x1.5mm, F.Cu at (86.0, 135.0)
- added TP27: GND, TestPoint:TestPoint_Pad_1.5x1.5mm, F.Cu at (80.0, 135.0)
- added TP28: PC7, TestPoint:TestPoint_Pad_1.5x1.5mm, F.Cu at (74.0, 135.0)
- added TP29: SWIO, TestPoint:TestPoint_Pad_1.5x1.5mm, F.Cu at (37.0, 135.0)
- added TP3: GND, TestPoint:TestPoint_Pad_1.5x1.5mm, F.Cu at (50.0, 30.0)
- added TP30: 3V3, TestPoint:TestPoint_Pad_1.5x1.5mm, F.Cu at (31.0, 135.0)
- added TP31: GND, TestPoint:TestPoint_Pad_1.5x1.5mm, F.Cu at (25.0, 135.0)
- added TP32: PC7, TestPoint:TestPoint_Pad_1.5x1.5mm, F.Cu at (19.0, 135.0)
- added TP4: PC7, TestPoint:TestPoint_Pad_1.5x1.5mm, F.Cu at (56.0, 30.0)
- added TP5: SWIO, TestPoint:TestPoint_Pad_1.5x1.5mm, F.Cu at (93.0, 30.0)
- added TP6: 3V3, TestPoint:TestPoint_Pad_1.5x1.5mm, F.Cu at (99.0, 30.0)
- added TP7: GND, TestPoint:TestPoint_Pad_1.5x1.5mm, F.Cu at (105.0, 30.0)
- added TP8: PC7, TestPoint:TestPoint_Pad_1.5x1.5mm, F.Cu at (111.0, 30.0)
- added TP9: SWIO, TestPoint:TestPoint_Pad_1.5x1.5mm, F.Cu at (148.0, 30.0)
- added U1: SN74LVC1G3157, Package_TO_SOT_SMD:SOT-23-6, F.Cu at (135.0, 90.0)
- added U10: 74HC595, Package_SO:SOIC-16_3.9x9.9mm_P1.27mm, F.Cu at (192.0, 73.0)
- added U100: CH32V003F4P6, Package_SO:TSSOP-20_4.4x6.5mm_P0.65mm, F.Cu at (147.5, 147.0)
- added U101: ADCS7476, Package_TO_SOT_SMD:SOT-23-6, F.Cu at (78.0, 146.0)
- added U102: INA241A5, Package_TO_SOT_SMD:SOT-23-8, F.Cu at (72.0, 146.0)
- added U103: DNP, Package_TO_SOT_SMD:SOT-23-5, F.Cu at (116.0, 153.0)
- added U104: SN74LVC1G3157, Package_TO_SOT_SMD:SOT-23-6, F.Cu at (109.0, 143.0)
- added U105: CH32V003F4P6, Package_SO:TSSOP-20_4.4x6.5mm_P0.65mm, F.Cu at (92.5, 147.0)
- added U106: 74LVC1G3157, Package_TO_SOT_SMD:SOT-23-6, F.Cu at (23.0, 150.0)
- added U107: 74LVC1G3157, Package_TO_SOT_SMD:SOT-23-6, F.Cu at (17.0, 150.0)
- added U108: 74LVC1G3157, Package_TO_SOT_SMD:SOT-23-6, F.Cu at (11.0, 150.0)
- added U109: 74LVC1G3157, Package_TO_SOT_SMD:SOT-23-6, F.Cu at (29.0, 154.0)
- added U11: 74HC165, Package_SO:SOIC-16_3.9x9.9mm_P1.27mm, F.Cu at (204.0, 73.0)
- added U110: 74LVC1G3157, Package_TO_SOT_SMD:SOT-23-6, F.Cu at (23.0, 154.0)
- added U111: 74LVC1G3157, Package_TO_SOT_SMD:SOT-23-6, F.Cu at (17.0, 154.0)
- added U112: 74LVC1G3157, Package_TO_SOT_SMD:SOT-23-6, F.Cu at (11.0, 154.0)
- added U113: 74LVC1G3157, Package_TO_SOT_SMD:SOT-23-6, F.Cu at (29.0, 158.0)
- added U114: DNP, Package_TO_SOT_SMD:SOT-23-5, F.Cu at (61.0, 153.0)
- added U115: SN74LVC1G3157, Package_TO_SOT_SMD:SOT-23-6, F.Cu at (54.0, 143.0)
- added U116: CH32V003F4P6, Package_SO:TSSOP-20_4.4x6.5mm_P0.65mm, F.Cu at (37.5, 147.0)
- added U12: 74HC165, Package_SO:SOIC-16_3.9x9.9mm_P1.27mm, F.Cu at (216.0, 73.0)
- added U13: 74HC595, Package_SO:SOIC-16_3.9x9.9mm_P1.27mm, F.Cu at (17.0, 61.0)
- added U14: 74HC595, Package_SO:SOIC-16_3.9x9.9mm_P1.27mm, F.Cu at (72.0, 61.0)
- added U15: 74HC595, Package_SO:SOIC-16_3.9x9.9mm_P1.27mm, F.Cu at (127.0, 61.0)
- added U16: 74HC595, Package_SO:SOIC-16_3.9x9.9mm_P1.27mm, F.Cu at (182.0, 61.0)
- added U17: 74HC595, Package_SO:SOIC-16_3.9x9.9mm_P1.27mm, F.Cu at (223.0, 166.0)
- added U18: 74HC595, Package_SO:SOIC-16_3.9x9.9mm_P1.27mm, F.Cu at (168.0, 166.0)
- added U19: 74HC595, Package_SO:SOIC-16_3.9x9.9mm_P1.27mm, F.Cu at (113.0, 166.0)
- added U2: SN74LVC1G3157, Package_TO_SOT_SMD:SOT-23-6, F.Cu at (145.0, 78.0)
- added U20: 74HC595, Package_SO:SOIC-16_3.9x9.9mm_P1.27mm, F.Cu at (58.0, 166.0)
- added U21: AMS1117-3.3, Package_TO_SOT_SMD:SOT-223-3_TabPin2, F.Cu at (22.0, 102.0)
- added U22: 74LVC1G3157, Package_TO_SOT_SMD:SOT-23-6, F.Cu at (40.0, 80.0)
- added U23: 74LVC1G3157, Package_TO_SOT_SMD:SOT-23-6, F.Cu at (46.0, 80.0)
- added U24: 74LVC1G3157, Package_TO_SOT_SMD:SOT-23-6, F.Cu at (34.0, 88.0)
- added U25: 74LVC1G3157, Package_TO_SOT_SMD:SOT-23-6, F.Cu at (40.0, 88.0)
- added U26: 74LVC1G3157, Package_TO_SOT_SMD:SOT-23-6, F.Cu at (46.0, 88.0)
- added U27: 74LVC1G3157, Package_TO_SOT_SMD:SOT-23-6, F.Cu at (34.0, 96.0)
- added U28: RP2040, Package_DFN_QFN:QFN-56-1EP_7x7mm_P0.4mm_EP3.2x3.2mm, F.Cu at (66.0, 90.0)
- added U29: W25Q16JVSSIQ, Package_SO:SOIC-8_5.3x5.3mm_P1.27mm, F.Cu at (79.0, 90.0)
- added U3: SN74LVC1G3157, Package_TO_SOT_SMD:SOT-23-6, F.Cu at (145.0, 102.0)
- added U30: SN74LVC1G3157, Package_TO_SOT_SMD:SOT-23-6, F.Cu at (96.0, 90.0)
- added U31: SN74LVC1G3157, Package_TO_SOT_SMD:SOT-23-6, F.Cu at (106.0, 78.0)
- added U32: SN74LVC1G3157, Package_TO_SOT_SMD:SOT-23-6, F.Cu at (106.0, 102.0)
- added U33: SN74LVC1G3157, Package_TO_SOT_SMD:SOT-23-6, F.Cu at (116.0, 70.0)
- added U34: SN74LVC1G3157, Package_TO_SOT_SMD:SOT-23-6, F.Cu at (116.0, 80.0)
- added U35: SN74LVC1G3157, Package_TO_SOT_SMD:SOT-23-6, F.Cu at (116.0, 100.0)
- added U36: SN74LVC1G3157, Package_TO_SOT_SMD:SOT-23-6, F.Cu at (116.0, 110.0)
- added U37: 74LVC1G3157, Package_TO_SOT_SMD:SOT-23-6, F.Cu at (46.0, 41.0)
- added U38: 74LVC1G3157, Package_TO_SOT_SMD:SOT-23-6, F.Cu at (52.0, 41.0)
- added U39: 74LVC1G3157, Package_TO_SOT_SMD:SOT-23-6, F.Cu at (58.0, 41.0)
- added U4: SN74LVC1G3157, Package_TO_SOT_SMD:SOT-23-6, F.Cu at (155.0, 70.0)
- added U40: 74LVC1G3157, Package_TO_SOT_SMD:SOT-23-6, F.Cu at (64.0, 41.0)
- added U41: 74LVC1G3157, Package_TO_SOT_SMD:SOT-23-6, F.Cu at (46.0, 45.0)
- added U42: 74LVC1G3157, Package_TO_SOT_SMD:SOT-23-6, F.Cu at (52.0, 45.0)
- added U43: 74LVC1G3157, Package_TO_SOT_SMD:SOT-23-6, F.Cu at (58.0, 45.0)
- added U44: 74LVC1G3157, Package_TO_SOT_SMD:SOT-23-6, F.Cu at (64.0, 45.0)
- added U45: DNP, Package_TO_SOT_SMD:SOT-23-5, F.Cu at (14.0, 48.0)
- added U46: SN74LVC1G3157, Package_TO_SOT_SMD:SOT-23-6, F.Cu at (21.0, 38.0)
- added U47: CH32V003F4P6, Package_SO:TSSOP-20_4.4x6.5mm_P0.65mm, F.Cu at (37.5, 42.0)
- added U48: 74LVC1G3157, Package_TO_SOT_SMD:SOT-23-6, F.Cu at (107.0, 45.0)
- added U49: 74LVC1G3157, Package_TO_SOT_SMD:SOT-23-6, F.Cu at (113.0, 45.0)
- added U5: SN74LVC1G3157, Package_TO_SOT_SMD:SOT-23-6, F.Cu at (155.0, 80.0)
- added U50: 74LVC1G3157, Package_TO_SOT_SMD:SOT-23-6, F.Cu at (119.0, 45.0)
- added U51: 74LVC1G3157, Package_TO_SOT_SMD:SOT-23-6, F.Cu at (101.0, 49.0)
- added U52: 74LVC1G3157, Package_TO_SOT_SMD:SOT-23-6, F.Cu at (107.0, 49.0)
- added U53: 74LVC1G3157, Package_TO_SOT_SMD:SOT-23-6, F.Cu at (113.0, 49.0)
- added U54: 74LVC1G3157, Package_TO_SOT_SMD:SOT-23-6, F.Cu at (119.0, 49.0)
- added U55: 74LVC1G3157, Package_TO_SOT_SMD:SOT-23-6, F.Cu at (101.0, 53.0)
- added U56: DNP, Package_TO_SOT_SMD:SOT-23-5, F.Cu at (69.0, 48.0)
- added U57: SN74LVC1G3157, Package_TO_SOT_SMD:SOT-23-6, F.Cu at (76.0, 38.0)
- added U58: CH32V003F4P6, Package_SO:TSSOP-20_4.4x6.5mm_P0.65mm, F.Cu at (92.5, 42.0)
- added U59: 74LVC1G3157, Package_TO_SOT_SMD:SOT-23-6, F.Cu at (174.0, 37.0)
- added U6: SN74LVC1G3157, Package_TO_SOT_SMD:SOT-23-6, F.Cu at (155.0, 100.0)
- added U60: 74LVC1G3157, Package_TO_SOT_SMD:SOT-23-6, F.Cu at (156.0, 41.0)
- added U61: 74LVC1G3157, Package_TO_SOT_SMD:SOT-23-6, F.Cu at (162.0, 41.0)
- added U62: 74LVC1G3157, Package_TO_SOT_SMD:SOT-23-6, F.Cu at (168.0, 41.0)
- added U63: 74LVC1G3157, Package_TO_SOT_SMD:SOT-23-6, F.Cu at (174.0, 41.0)
- added U64: 74LVC1G3157, Package_TO_SOT_SMD:SOT-23-6, F.Cu at (156.0, 45.0)
- added U65: 74LVC1G3157, Package_TO_SOT_SMD:SOT-23-6, F.Cu at (162.0, 45.0)
- added U66: DNP, Package_TO_SOT_SMD:SOT-23-5, F.Cu at (124.0, 48.0)
- added U67: SN74LVC1G3157, Package_TO_SOT_SMD:SOT-23-6, F.Cu at (131.0, 38.0)
- added U68: CH32V003F4P6, Package_SO:TSSOP-20_4.4x6.5mm_P0.65mm, F.Cu at (147.5, 42.0)
- added U69: 74LVC1G3157, Package_TO_SOT_SMD:SOT-23-6, F.Cu at (217.0, 45.0)
- added U7: SN74LVC1G3157, Package_TO_SOT_SMD:SOT-23-6, F.Cu at (155.0, 110.0)
- added U70: 74LVC1G3157, Package_TO_SOT_SMD:SOT-23-6, F.Cu at (223.0, 45.0)
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Other:
- board outline added: 240 x 180 mm
- board text added: "AUX0"
- board text added: "AUX1"
- board text added: "AUX2"
- board text added: "OBS0"
- board text added: "OBS1"
- board text added: "T0"
- board text added: "T1"
- board text added: "T2"
- board text added: "T3"
- board text added: "T4"
- board text added: "T5"
- board text added: "T6"
- board text added: "T7"
